File: documents/schematics/baseboard.sch (EAGLE design)
At the start: 16 parts, among them Q1 20 MHz, Q2 BS170, Q3 BS170, T1 2N3904

Commit message: Baseboard getting bigger and bigger
Parts:
- added C10, C8: 0,1µF, capacitor-wima:C2.5/2
- added C11, C5, C9: 10µF, capacitor-wima:C2.5/2
- added C12: 22pF, capacitor-wima:C2.5/2
- added C13: 22pf, capacitor-wima:C2.5/2
- added C6: 100nF, capacitor-wima:C2.5/2
- added C7: 220µF, capacitor-wima:C2.5/2
- added D1: 1N4004, diode:1N4004
- added IC1: MAX 603, ic-package:DIL8
- added IC2: AD780N, analog-devices:AD780N
- added J1: 350792-1, con-amp:350792-1
- added Q4: 5 MHz, crystal:CRYSTALHC49S
- added R5: 22k, resistor:R-EU_0207/2V
- added R6: 1.1k, resistor:R-EU_0207/2V
- added R7: 20k, resistor:R-EU_0207/2V
- added R8: 2.2k, resistor:R-EU_0207/2V
- added TB1, TB6560: (no value), con-ml:ML10
- added U$3: AD7705, AD7705:AD7705
Connections:
- removed net VCC: C1.2, JP1.2, R1.1, R2.2, R3.2, T1.C, U$1.VCC
- new net +3V3: C5.2, C8.2, C9.2, IC1.8, J1.4, U$3.RESET, U$3.VDD
- new net +5V: C1.2, D1.A, IC2.+VIN, J1.1, JP1.2, R1.1, R2.2, R3.2, T1.C, U$1.VCC
- new net N$23: TB6560.10, U$1.(ICP)PD6
- new net N$24: GPIO.12, TB1.9
- new net N$25: GPIO.10, TB1.7
- new net N$26: GPIO.8, TB1.5
- new net N$27: GPIO.23, TB1.10
- new net N$29: GPIO.21, TB1.8
- new net N$30: GPIO.19, TB1.6
- new net N$31: C10.2, C11.2, IC2.VOUT, U$3.REF+
- new net N$32: C6.2, C7.2, D1.C, IC1.1, IC1.4
- new net N$35: C12.2, Q4.2, U$3.MCLKIN
- new net N$36: C13.2, Q4.1, U$3.MCLKOUT
- new net N$37: R5.1, R6.1, U$3.AIN2+
- new net N$38: R7.1, R8.1, U$3.AIN1+
- net GND: now also C10.1, C11.1, C12.1, C13.1, C5.1, C6.1, C7.1, C8.1, C9.1, IC1.2, IC1.3, IC1.5, IC1.6, IC1.7, IC2.GND, J1.2, J1.3, R6.2, R8.2, U$3.AIN1-, U$3.AIN2-, U$3.GND, U$3.REF-
- net N$10: now also TB6560.3, U$1.(OC1A)PB3; no longer U$1.(AIN1)PB1
- net N$11: now also TB6560.1, U$1.(OC1B)PB4; no longer U$1.(AIN0)PB0
- net N$12: now also TB6560.4, U$1.(TXD)PD1; no longer U$1.(ICP)PD6
- net N$13: now also TB6560.6, U$1.(T0)PD4; no longer U$1.(TXD)PD1
- net N$14: now also TB6560.8, U$1.(T1)PD5; no longer U$1.(RXD)PD0
- net N$16: now also TB1.1
- net N$2: now also TB1.3
- net N$28: now also TB1.2
- net N$4: now also TB1.4
- net N$6: now also TB6560.2, U$1.(RXD)PD0; no longer U$1.(T1)PD5
- net N$7: now also TB6560.9, U$1.(AIN0)PB0; no longer U$1.(OC0A)PB2
- net N$8: now also TB6560.7, U$1.(AIN1)PB1; no longer U$1.(OC1A)PB3
- net N$9: now also TB6560.5, U$1.(OC0A)PB2; no longer U$1.(OC1B)PB4
Other:
- note removed: "X-CLK (step)"
- note removed: "X-CW/CCW (direction)"
- note removed: "X-ENABLE"
- note removed: "Y-CLK (step)"
- note removed: "Y-CW/CCW (direction)"
- note removed: "Y-ENABLE"
- note removed: "Z-CLK (step)"
- note removed: "Z-CW/CCW (direction)"
- note removed: "Z-ENABLE"
- moved on the sheet: C4, GPIO, JP1, Q2, Q3, R2, R3, R4, T1

Commit message: Changed label of MAX 604
Parts:
- IC1: value MAX 603 -> MAX 604
Changed lines of the file:
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@@
 <part name="TB1" library="con-ml" deviceset="ML10" device=""/>
 <part name="J1" library="con-amp" deviceset="350792-1" device=""/>
-<part name="IC1" library="ic-package" deviceset="DIL8" device="" value="MAX 603"/>
+<part name="IC1" library="ic-package" deviceset="DIL8" device="" value="MAX 604"/>
 <part name="C5" library="capacitor-wima" deviceset="C" device="2.5/2" value="10µF"/>
 <part name="C6" library="capacitor-wima" deviceset="C" device="2.5/2" value="100nF"/>

Commit message: Baseboard alpha
Parts:
- added JP2: 12.6V LiPo, pinhead:PINHD-1X2
- added JP3: 25.2V LiPo, pinhead:PINHD-1X2
Connections:
- new net N$33: JP3.1, R6.2
- new net N$34: JP2.1, R8.2
- new net N$39: JP3.2, R5.2
- new net N$42: GPIO.14, U$3.DRDY
- new net N$43: GPIO.16, U$3.RESET
- net +3V3: no longer U$3.RESET
- net GND: no longer R6.2, R8.2
- net N$27: now also U$3.SCLK
- net N$29: now also U$3.DOUT
- net N$30: now also U$3.DIN
- net N$32: now also JP2.2, R7.2
Other:
- moved on the sheet: C1, C10, C11, C12, C13, C2, C3, C4, C5, C6, C7, C8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

Commit message: Baseboard Bugfix
Connections:
- removed net N$42: GPIO.14, U$3.DRDY
- new net N$40: GPIO.22, U$3.DRDY
- new net N$41: GPIO.16, U$3.CS
- net N$43: now also GPIO.18; no longer GPIO.16
Other:
- moved on the sheet: C1, C10, C11, C12, C13, C2, C3, C4, C5, C6, C7, C8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

Commit message: Updated schematics
Connections:
- removed net N$14 (its old number): TB6560.8, U$1.(T1)PD5
- removed net N$23 (its old number): TB6560.10, U$1.(ICP)PD6
- new net N$12: TB6560.8, U$1.(AIN0)PB0
- new net N$6: TB6560.1, U$1.(T0)PD4
- net N$10: now also TB6560.9, U$1.(OC0A)PB2; no longer TB6560.3, U$1.(OC1A)PB3
- net N$11: now also TB6560.10, U$1.(AIN1)PB1; no longer TB6560.1, U$1.(OC1B)PB4
- net N$13: now also U$1.(ICP)PD6; no longer U$1.(T0)PD4
- net N$7: now also TB6560.3, U$1.(T1)PD5; no longer TB6560.9, U$1.(AIN0)PB0
- net N$8: now also TB6560.5, U$1.(OC1B)PB4; no longer TB6560.7, U$1.(AIN1)PB1
- net N$9: now also TB6560.7, U$1.(OC1A)PB3; no longer TB6560.5, U$1.(OC0A)PB2
Changed lines of the file:
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@@
-</segment>
-</net>
-<net name="N$7" class="0">
-<segment>
-<pinref part="U$1" gate="G$1" pin="(AIN0)PB0"/>
-<pinref part="TB6560" gate="G$1" pin="9"/>
-<wire x1="170.18" y1="48.26" x2="185.42" y2="48.26" width="0.1524" layer="91"/>
-<wire x1="185.42" y1="48.26" x2="185.42" y2="25.4" width="0.1524" layer="91"/>
-</segment>
-</net>
-<net name="N$8" class="0">
-<segment>
-<pinref part="U$1" gate="G$1" pin="(AIN1)PB1"/>
-<pinref part="TB6560" gate="G$1" pin="7"/>
-<wire x1="170.18" y1="50.8" x2="187.96" y2="50.8" width="0.1524" layer="91"/>
-<wire x1="187.96" y1="50.8" x2="187.96" y2="25.4" width="0.1524" layer="91"/>
-</segment>
-</net>
-<net name="N$9" class="0">
-<segment>
-<pinref part="U$1" gate="G$1" pin="(OC0A)PB2"/>
-<pinref part="TB6560" gate="G$1" pin="5"/>
-<wire x1="170.18" y1="53.34" x2="190.5" y2="53.34" width="0.1524" layer="91"/>
-<wire x1="190.5" y1="53.34" x2="190.5" y2="25.4" width="0.1524" layer="91"/>
-</segment>
-</net>
-<net name="N$10" class="0">
-<segment>
-<pinref part="U$1" gate="G$1" pin="(OC1A)PB3"/>
-<pinref part="TB6560" gate="G$1" pin="3"/>
-<wire x1="170.18" y1="55.88" x2="193.04" y2="55.88" width="0.1524" layer="91"/>
-<wire x1="193.04" y1="55.88" x2="193.04" y2="25.4" width="0.1524" layer="91"/>
-</segment>
-</net>
-<net name="N$11" class="0">
-<segment>
-<pinref part="U$1" gate="G$1" pin="(OC1B)PB4"/>
-<pinref part="TB6560" gate="G$1" pin="1"/>
-<wire x1="170.18" y1="58.42" x2="195.58" y2="58.42" width="0.1524" layer="91"/>
-<wire x1="195.58" y1="58.42" x2="195.58" y2="25.4" width="0.1524" layer="91"/>
-</segment>
-</net>
-<net name="N$6" class="0">
-<segment>
-<pinref part="U$1" gate="G$1" pin="(RXD)PD0"/>
-<wire x1="170.18" y1="22.86" x2="170.18" y2="0" width="0.1524" layer="91"/>
-<pinref part="TB6560" gate="G$1" pin="2"/>
-<wire x1="170.18" y1="0" x2="195.58" y2="0" width="0.1524" layer="91"/>
-<wire x1="195.58" y1="0" x2="195.58" y2="10.16" width="0.1524" layer="91"/>
-</segment>
-</net>
-<net name="N$12" class="0">
-<segment>
-<pinref part="U$1" gate="G$1" pin="(TXD)PD1"/>
-<wire x1="170.18" y1="25.4" x2="172.72" y2="25.4" width="0.1524" layer="91"/>
-<wire x1="172.72" y1="25.4" x2="172.72" y2="2.54" width="0.1524" layer="91"/>
-<pinref part="TB6560" gate="G$1" pin="4"/>
-<wire x1="172.72" y1="2.54" x2="193.04" y2="2.54" width="0.1524" layer="91"/>
-<wire x1="193.04" y1="2.54" x2="193.04" y2="10.16" width="0.1524" layer="91"/>
-</segment>
-</net>
-<net name="N$13" class="0">
-<segment>
-<pinref part="TB6560" gate="G$1" pin="6"/>
-<wire x1="190.5" y1="10.16" x2="190.5" y2="5.08" width="0.1524" layer="91"/>
-<wire x1="190.5" y1="5.08" x2="175.26" y2="5.08" width="0.1524" layer="91"/>
-<wire x1="175.26" y1="5.08" x2="175.26" y2="33.02" width="0.1524" layer="91"/>
-<pinref part="U$1" gate="G$1" pin="(T0)PD4"/>
-<wire x1="175.26" y1="33.02" x2="170.18" y2="33.02" width="0.1524" layer="91"/>
-</segment>
-</net>
-<net name="N$14" class="0">
-<segment>
-<pinref part="U$1" gate="G$1" pin="(T1)PD5"/>
-<wire x1="170.18" y1="35.56" x2="177.8" y2="35.56" width="0.1524" layer="91"/>
-<wire x1="177.8" y1="35.56" x2="177.8" y2="7.62" width="0.1524" layer="91"/>
-<wire x1="177.8" y1="7.62" x2="187.96" y2="7.62" width="0.1524" layer="91"/>
-<pinref part="TB6560" gate="G$1" pin="8"/>
-<wire x1="187.96" y1="7.62" x2="187.96" y2="10.16" width="0.1524" layer="91"/>
-</segment>
-</net>
-<net name="N$23" class="0">
-<segment>
-<pinref part="TB6560" gate="G$1" pin="10"/>
-<wire x1="185.42" y1="10.16" x2="180.34" y2="10.16" width="0.1524" layer="91"/>
-<wire x1="180.34" y1="10.16" x2="180.34" y2="38.1" width="0.1524" layer="91"/>
-<pinref part="U$1" gate="G$1" pin="(ICP)PD6"/>
-<wire x1="180.34" y1="38.1" x2="170.18" y2="38.1" width="0.1524" layer="91"/>
 </segment>
 </net>
@@
 </segment>
 </net>
+<net name="N$6" class="0">
+<segment>
+<pinref part="TB6560" gate="G$1" pin="1"/>
+<wire x1="195.58" y1="25.4" x2="195.58" y2="33.02" width="0.1524" layer="91"/>
+<pinref part="U$1" gate="G$1" pin="(T0)PD4"/>
+<wire x1="195.58" y1="33.02" x2="170.18" y2="33.02" width="0.1524" layer="91"/>
+</segment>
+</net>
+<net name="N$7" class="0">
+<segment>
+<pinref part="TB6560" gate="G$1" pin="3"/>
+<wire x1="193.04" y1="25.4" x2="193.04" y2="35.56" width="0.1524" layer="91"/>
+<pinref part="U$1" gate="G$1" pin="(T1)PD5"/>
+<wire x1="193.04" y1="35.56" x2="170.18" y2="35.56" width="0.1524" layer="91"/>
+</segment>
+</net>
+<net name="N$8" class="0">
+<segment>
+<pinref part="TB6560" gate="G$1" pin="5"/>
+<wire x1="190.5" y1="25.4" x2="190.5" y2="58.42" width="0.1524" layer="91"/>
+<pinref part="U$1" gate="G$1" pin="(OC1B)PB4"/>
+<wire x1="190.5" y1="58.42" x2="170.18" y2="58.42" width="0.1524" layer="91"/>
+</segment>
+</net>
+<net name="N$9" class="0">
+<segment>
+<pinref part="TB6560" gate="G$1" pin="7"/>
+<wire x1="187.96" y1="25.4" x2="187.96" y2="55.88" width="0.1524" layer="91"/>
+<pinref part="U$1" gate="G$1" pin="(OC1A)PB3"/>
+<wire x1="187.96" y1="55.88" x2="170.18" y2="55.88" width="0.1524" layer="91"/>
+</segment>
+</net>
+<net name="N$10" class="0">
+<segment>
+<pinref part="TB6560" gate="G$1" pin="9"/>
+<wire x1="185.42" y1="25.4" x2="185.42" y2="53.34" width="0.1524" layer="91"/>
+<pinref part="U$1" gate="G$1" pin="(OC0A)PB2"/>
+<wire x1="185.42" y1="53.34" x2="170.18" y2="53.34" width="0.1524" layer="91"/>
+</segment>
+</net>
+<net name="N$11" class="0">
+<segment>
+<pinref part="TB6560" gate="G$1" pin="10"/>
+<wire x1="185.42" y1="10.16" x2="185.42" y2="7.62" width="0.1524" layer="91"/>
+<wire x1="185.42" y1="7.62" x2="180.34" y2="7.62" width="0.1524" layer="91"/>
+<wire x1="180.34" y1="7.62" x2="180.34" y2="50.8" width="0.1524" layer="91"/>
+<pinref part="U$1" gate="G$1" pin="(AIN1)PB1"/>
+<wire x1="180.34" y1="50.8" x2="170.18" y2="50.8" width="0.1524" layer="91"/>
+</segment>
+</net>
+<net name="N$12" class="0">
+<segment>
+<pinref part="TB6560" gate="G$1" pin="8"/>
+<wire x1="187.96" y1="10.16" x2="187.96" y2="5.08" width="0.1524" layer="91"/>
+<wire x1="187.96" y1="5.08" x2="177.8" y2="5.08" width="0.1524" layer="91"/>
+<wire x1="177.8" y1="5.08" x2="177.8" y2="48.26" width="0.1524" layer="91"/>
+<pinref part="U$1" gate="G$1" pin="(AIN0)PB0"/>
+<wire x1="177.8" y1="48.26" x2="170.18" y2="48.26" width="0.1524" layer="91"/>
+</segment>
+</net>
+<net name="N$13" class="0">
+<segment>
+<pinref part="TB6560" gate="G$1" pin="6"/>
+<wire x1="190.5" y1="10.16" x2="190.5" y2="2.54" width="0.1524" layer="91"/>
+<wire x1="190.5" y1="2.54" x2="175.26" y2="2.54" width="0.1524" layer="91"/>
+<wire x1="175.26" y1="2.54" x2="175.26" y2="38.1" width="0.1524" layer="91"/>
+<pinref part="U$1" gate="G$1" pin="(ICP)PD6"/>
+<wire x1="175.26" y1="38.1" x2="170.18" y2="38.1" width="0.1524" layer="91"/>
+</segment>
+</net>
+<net name="N$14" class="0">
+<segment>
+<pinref part="TB6560" gate="G$1" pin="4"/>
+<wire x1="193.04" y1="10.16" x2="193.04" y2="0" width="0.1524" layer="91"/>
+<wire x1="193.04" y1="0" x2="172.72" y2="0" width="0.1524" layer="91"/>
+<wire x1="172.72" y1="0" x2="172.72" y2="25.4" width="0.1524" layer="91"/>
+<pinref part="U$1" gate="G$1" pin="(TXD)PD1"/>
+<wire x1="172.72" y1="25.4" x2="170.18" y2="25.4" width="0.1524" layer="91"/>
+</segment>
+</net>
+<net name="N$23" class="0">
+<segment>
+<pinref part="U$1" gate="G$1" pin="(RXD)PD0"/>
+<wire x1="170.18" y1="22.86" x2="170.18" y2="-2.54" width="0.1524" layer="91"/>
+<pinref part="TB6560" gate="G$1" pin="2"/>
+<wire x1="170.18" y1="-2.54" x2="195.58" y2="-2.54" width="0.1524" layer="91"/>
+<wire x1="195.58" y1="-2.54" x2="195.58" y2="10.16" width="0.1524" layer="91"/>
+</segment>
+</net>
